Commit message: not final yet

File: ROS_ownpack/src/atom/urdf/atom.xacro (robot description, xacro)
@@ -157,4 +157,28 @@
 		</collision>
 	</link>
+	<!-- Hokuyo Lidar -->
+	<link name="hokuyo">
+		<inertial>
+			<mass value="${hokoyu_mass}"/>
+			<origin xyz="0 0 0" rpy="0 0 0"/>
+			<inertia
+		        ixx="1e-6" ixy="0.0" ixz="0.0"
+		        iyy="1e-6" iyz="0.0"
+		        izz="1e-6"
+		      />
+		</inertial>
+		<visual>
+			<origin xyz="0 0 0" rpy="0 0 0"/>
+			<geometry>
+				<mesh filename="package://atom/meshes/hokuyo.dae"/>
+			</geometry>
+		</visual>
+		<collision>
+			<origin xyz="0 0 0" rpy="0 0 0"/>
+			<geometry>
+				<box size="0.1 0.1 0.1"/>
+			</geometry>
+		</collision>
+	</link>
 	<!-- Project center to the ground -->
 	<link name="robot_footprint"></link>
@@ -203,4 +227,16 @@
 		<axis xyz="0 1 0"/>
 	</joint>
+	<!-- Hokoyu Joint -->
+	<joint name="hokuyo_joint" type="fixed">
+	    <origin xyz="0.2 0 0.2" rpy="0 0 0" />
+	    <parent link="chassis"/>
+	    <child link="hokuyo" />
+	    <axis xyz="0 1 0"/>
+	</joint>
+	<joint name="robot_footprint_joint" type="fixed">
+		<origin xyz="0 0 0" rpy="0 0 0" />
+		<parent link="robot_footprint"/>
+		<child link="chassis" />
+	</joint>
 	<!-- Color of bot -->
 	<gazebo reference="left_wheel_front">
